File: lily.kicad_pcb (KiCad board)
At the start: 4 copper layers, 70.7 x 53.3 mm, 31 parts, among them J1 NEIGHBOR1, J10 TEST_2P, J11 Conn_01x02, J12 TEST_2P, J13 TEST_2P, J14 TEST_2P, J15 TEST_2P, J16 TEST_2P, J17 TEST_2P, J18 TEST_2P, J2 NEIGHBOR2, J3 ANT_IN, J4 TEST_2P, J5 TEST_2P, J6 TEST_2P, J7 BONUS_ROW, J8 TEST_2P, J9 TEST_2P, U1 ADL5904

Commit message: adopt OSHWA convention for SPI signal names https://www.oshwa.org/a-resolution-to-redefine-spi-signal-names
Other:
- board text added: "CIPO"
- board text added: "COPI"
- board text added: "CS"
- board text removed: "MISO"
- board text removed: "MOSI"
- board text removed: "SSEL"
Changed lines of the file:
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@@
     (effects (font (size 0.635 0.508) (thickness 0.1016)))
   )
-  (gr_text SSEL (at 167.64 121.412) (layer F.SilkS)
+  (gr_text CS (at 167.64 121.412) (layer F.SilkS)
     (effects (font (size 0.635 0.508) (thickness 0.1016)))
   )
-  (gr_text MISO (at 172.72 116.84) (layer F.SilkS)
+  (gr_text CIPO (at 172.72 116.84) (layer F.SilkS)
     (effects (font (size 0.635 0.508) (thickness 0.1016)))
   )
-  (gr_text MOSI (at 172.72 119.38) (layer F.SilkS)
+  (gr_text COPI (at 172.72 119.38) (layer F.SilkS)
     (effects (font (size 0.635 0.508) (thickness 0.1016)))
   )
